File: keyboard.kicad_pcb (KiCad board)
At the start: 2 copper layers, 75.4 x 113.7 mm, 79 parts, among them IC1 ATMEGA32U4, J1 MINI, P1 MISO, P2 Vcc, P200 GND, P201 GND, P202 GND, P203 GND, P3 SCK, P4 MOSI, P5 RES, P6 GND, X1 ASX3F

Commit message: v0.2
Parts:
- added D23: 1N4148, SM0805D, B.Cu at (114.6, 175.4)
- added D24: 1N4148, SM0805D, B.Cu at (133.7, 175.4)
- added P204: GND, Pad-Gnd, F.Cu at (136.8, 177.3)
- added P205: GND, Pad-Gnd, F.Cu at (63.2, 177.3)
- added P300: DRL, Pad_Drl, B.Cu at (100.0, 159.4)
- added P301: DRL, Pad_Drl, B.Cu at (102.4, 159.4)
- added P302: DRL, Pad_Drl, B.Cu at (105.0, 159.4)
- added S171: MX1A, CHERRY_PCB_200H_Visible, F.Cu at (128.6, 102.4)
- added S181: MX1A, CHERRY_PCB_200H_Visible, F.Cu at (128.6, 121.4)
- added S191: MX1A, CHERRY_PCB_200H_Visible, F.Cu at (128.6, 140.5)
- added S201: MX1A, CHERRY_PCB_200H_Visible, F.Cu at (128.6, 159.5)
- added S211: MX1A, CHERRY_PCB_200H_Visible, F.Cu at (81.0, 169.1)
- added S23: MX1A, CHERRY_PCB_100H_Plated, F.Cu at (109.5, 169.1)
- added S24: MX1A, CHERRY_PCB_100H_Plated, F.Cu at (128.6, 169.1)
- added S51: MX1A, CHERRY_PCB_200H_Visible, F.Cu at (81.0, 150.0)
- S17, S18: footprint CHERRY_PCB_200H_Visible -> CHERRY_PCB_100H_Plated
- moved D19 70.1 mm to (134.9, 136.7), turned to 0 degrees
- moved S19 68.7 mm to (128.6, 131.0)
- moved P6 57.3 mm to (80.6, 104.6), turned to 90 degrees
- moved P1 54.1 mm to (80.6, 107.2), turned to 90 degrees
- moved P2 51.1 mm to (80.6, 109.7), turned to 90 degrees
- moved P3 48.1 mm to (80.6, 112.2), turned to 90 degrees
- moved P4 45.2 mm to (80.6, 114.8), turned to 90 degrees
- moved D20 44.0 mm to (134.9, 155.7), turned to 0 degrees
- moved S20 42.6 mm to (128.6, 150.0)
- moved P5 42.4 mm to (80.6, 117.3), turned to 90 degrees
- moved D21 40.7 mm to (74.0, 176.7), turned to 0 degrees
- moved S21 38.1 mm to (71.4, 169.1)
- moved S22 38.1 mm to (90.5, 169.1)
- moved D22 36.2 mm to (97.5, 176.7)
- moved S18 28.6 mm to (128.6, 111.9), turned to 180 degrees
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Connections:
- D17 pad 1: /Matrix/col4 -> N-0000055
- D17 pad 2: N-0000051 (its old number) -> /Matrix/col4
- D18 pad 1: /Matrix/col4 -> N-0000050
- D18 pad 2: N-0000045 -> /Matrix/col4
- D19 pad 1: /Matrix/col1 -> N-0000053
- D19 pad 2: N-0000055 -> /Matrix/col4
- D20 pad 1: /Matrix/col2 -> N-0000052
- D20 pad 2: N-0000053 -> /Matrix/col4
- D21 pad 1: /Matrix/col3 -> /Matrix/col1
- D22 pad 1: /Matrix/col4 -> /Matrix/col2
- D5 pad 1: /Matrix/col1 -> N-0000054
- D5 pad 2: N-0000047 (its old number) -> /Matrix/col1
- S17 pad 2: N-0000051 (its old number) -> N-0000055
- S18 pad 1: /Matrix/row4 -> /Matrix/row3
- S18 pad 2: N-0000045 -> N-0000050
- S19 pad 1: /Matrix/row6 -> /Matrix/row4
- S19 pad 2: N-0000055 -> N-0000053
- S20 pad 1: /Matrix/row6 -> /Matrix/row5
- S20 pad 2: N-0000053 -> N-0000052
- S5 pad 2: N-0000047 (its old number) -> N-0000054
Routing:
- net /Matrix/col1: track 205.0 -> 130.9 mm, vias 2 -> 3
- net /Matrix/row2: track 116.3 -> 170.9 mm
- net /Matrix/numlock: track 91.9 -> 52.4 mm, vias 1 -> 0
- net /Matrix/row3: track 49.8 -> 81.3 mm, vias 2 -> 1
- net GND: track 438.1 -> 407.2 mm, vias 1 -> 3
- net /~RES~: track 103.7 -> 74.7 mm
- net N-000006: track 86.9 -> 63.1 mm
- net /Matrix/row1: track 105.2 -> 126.8 mm
- net N-000001: track 58.0 -> 38.3 mm, vias 4 -> 2
- net /SCK: track 39.5 -> 20.2 mm, vias 1 -> 0
- net /MISO: track 42.7 -> 24.6 mm, vias 2 -> 1
- net /Matrix/col2: track 107.6 -> 123.7 mm
- net N-000008: track 25.0 -> 10.2 mm
- net /Matrix/row6: track 130.0 -> 116.0 mm
- net N-0000054: track 0.00 -> 13.3 mm
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Other:
- net class Default: clearance 0.2032 -> 0.2; trace_width 0.4064 -> 0.2
- net class POWER: clearance 0.2032 -> 0.2
- rule trace_clearance: 0.2032 -> 0.2
- rule trace_min: 0.2032 -> 0.2

Commit message: v0.3
Parts:
- added P303: DRL, Pad_Drl, B.Cu at (109.0, 159.4)
- added P304: DRL, Pad_Drl, B.Cu at (112.1, 159.4)
- added P305: DRL, Pad_Drl, B.Cu at (116.9, 159.4)
- added P306: DRL, Pad_Drl, B.Cu at (119.7, 159.4)
- added P307: DRL, Pad_Drl, B.Cu at (122.7, 159.4)
- added P309: DRL, Pad_Drl, B.Cu at (134.2, 159.4)
- added P310: DRL, Pad_Drl, B.Cu at (96.6, 159.4)
- added P311: DRL, Pad_Drl, B.Cu at (89.5, 159.4)
- added P312: DRL, Pad_Drl, B.Cu at (86.4, 159.4)
- added P313: DRL, Pad_Drl, B.Cu at (83.4, 159.4)
- added P314: DRL, Pad_Drl, B.Cu at (80.1, 159.4)
- added P315: DRL, Pad_Drl, B.Cu at (77.0, 159.4)
- added P316: DRL, Pad_Drl, B.Cu at (72.2, 159.4)
- added P317: DRL, Pad_Drl, B.Cu at (65.1, 159.4)
- moved P302 1.02 mm to (106.0, 159.4)
- moved P301 0.51 mm to (102.9, 159.4)

Commit message: v0.4
Parts:
- added H0: hole, PKRH, F.Cu at (100.0, 89.1)
- added H1: hole, PKRH, F.Cu at (100.0, 146.2)
- added P318: DRL, Pad_Drl, B.Cu at (62.8, 159.4)
- added P319: DRL, Pad_Drl, B.Cu at (137.2, 159.4)
- RF1, RF2, RF3: moved to B.Cu
- moved D21 13.7 mm to (79.1, 164.0)
- moved S0 1.91 mm to (100.0, 73.8), turned to 270 degrees
- moved D22 1.27 mm to (97.5, 175.4)
- moved P200 1.27 mm to (63.2, 157.0)
- moved D5 0.93 mm to (74.4, 155.5), turned to 270 degrees
- moved P202 0.64 mm to (136.8, 157.6)
- moved P317 0.38 mm to (65.5, 159.4)
- moved D6 0.38 mm to (95.2, 80.2)
- moved D20 0.13 mm to (134.8, 155.7)
- turned S21 to 0 degrees
- turned S5 to 0 degrees
Routing:
- net /Matrix/col2: track 123.7 -> 275.9 mm
- net GND: track 407.2 -> 534.5 mm, vias 3 -> 28
- net /Matrix/row2: track 170.9 -> 100.6 mm, vias 0 -> 1
- net /Matrix/col3: track 118.9 -> 170.1 mm, vias 2 -> 6
- net VCC: track 265.9 -> 314.6 mm, vias 2 -> 6
- net N-000001: track 38.3 -> 86.2 mm, vias 2 -> 5
- net N-000003: track 13.4 -> 55.4 mm
- net N-000002: track 53.1 -> 94.2 mm, vias 2 -> 6
- net /Matrix/col1: track 130.9 -> 172.0 mm
- net /Matrix/row3: track 81.3 -> 112.2 mm
- net /Matrix/col4: track 137.2 -> 159.2 mm, vias 0 -> 4
- net /Matrix/row1: track 126.8 -> 107.3 mm
- net /Matrix/row5: track 113.9 -> 133.3 mm, vias 1 -> 0
- net /Matrix/row6: track 116.0 -> 135.3 mm
- net /GPIO0: track 45.0 -> 63.6 mm
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