File: keyboard.sch (KiCad schematic (older format))
At the start: 32 parts, among them IC1 ATMEGA32U4, J1 MINI, P1 MISO, P2 Vcc, P200 GND, P201 GND, P202 GND, P203 GND, P3 SCK, P4 MOSI, P5 RES, P6 GND, X1 ASX3F

Commit message: v0.2
Parts:
- added P204, P205: GND, symbol CONN_1
Connections:
- net GND: now also P204.1, P205.1
Changed lines of the file:
@@
-EESchema Schematic File Version 2  date 9/17/2013 2:51:05 PM
+EESchema Schematic File Version 2  date 9/17/2013 3:48:13 PM
 LIBS:power
 LIBS:mx1a-simple
@@
 	10250 4550 10100 4550
 Connection ~ 10850 4550
+$Comp
+L CONN_1 P204
+U 1 1 5238B3AB
+P 5900 2600
+F 0 "P204" H 5980 2600 40  0000 L CNN
+F 1 "GND" H 5900 2655 30  0001 C CNN
+F 2 "" H 5900 2600 60  0001 C CNN
+F 3 "" H 5900 2600 60  0001 C CNN
+	1    5900 2600
+	1    0    0    -1
+$EndComp
+$Comp
+L CONN_1 P205
+U 1 1 5238B3B1
+P 5900 2700
+F 0 "P205" H 5980 2700 40  0000 L CNN
+F 1 "GND" H 5900 2755 30  0001 C CNN
+F 2 "" H 5900 2700 60  0001 C CNN
+F 3 "" H 5900 2700 60  0001 C CNN
+	1    5900 2700
+	1    0    0    -1
+$EndComp
+Wire Wire Line
+	5750 2600 5650 2600
+Wire Wire Line
+	5650 2700 5750 2700
 $EndSCHEMATC

Commit message: v0.8
Parts:
- added H2, M1, M10, M11, M12, M13, M14, M15, M16, M17, M2, M3, M4, M5, M6, M7, M8, M9: HOLE, ~, symbol ANYTHING
- added LOGO1: Geekhack, ~, symbol ANYTHING
- added P10: ROW4, symbol CONN_1
- added P11: ROW5, symbol CONN_1
- added P12: ROW6, symbol CONN_1
- added P13: COL1, symbol CONN_1
- added P14: COL2, symbol CONN_1
- added P15: COL3, symbol CONN_1
- added P16: COL4, symbol CONN_1
- added P17: FNLED, symbol CONN_1
- added P18: Vcc, symbol CONN_1
- added P19: GND, symbol CONN_1
- added P7: ROW1, symbol CONN_1
- added P8: ROW2, symbol CONN_1
- added P9: ROW3, symbol CONN_1
Connections:
- net GND: now also H2.0 (GND), LOGO1.0 (GND), M1.0 (GND), M10.0 (GND), M11.0 (GND), M12.0 (GND), M13.0 (GND), M14.0 (GND), M15.0 (GND), M16.0 (GND), M17.0 (GND), M2.0 (GND), M3.0 (GND), M4.0 (GND), M5.0 (GND), M6.0 (GND), M7.0 (GND), M8.0 (GND), M9.0 (GND), P19.1
- net MOSI: now also P17.1
- net VCC: now also P18.1
- net col1: now also P13.1
- net col2: now also P14.1
- net col3: now also P15.1
- net col4: now also P16.1
- net row1: now also P7.1
- net row2: now also P8.1
- net row3: now also P9.1
- net row4: now also P10.1
- net row5: now also P11.1
- net row6: now also P12.1

Commit message: v0.9
Parts:
- added H1, H3, H4, H5: HOLE, ~, symbol ANYTHING
Connections:
- net GND: now also H1.0 (GND), H3.0 (GND), H4.0 (GND), H5.0 (GND)
Other:
- moved on the sheet: H2, LOGO1
Changed lines of the file:
@@
-EESchema Schematic File Version 2  date 10/17/2013 12:48:39 PM
+EESchema Schematic File Version 2  date 10/20/2013 1:26:13 PM
 LIBS:power
 LIBS:mx1a-simple
@@
 Sheet 1 2
 Title "4x6 keypad"
-Date "17 oct 2013"
-Rev "0.8"
+Date "20 oct 2013"
+Rev "0.9"
 Comp "regack"
 Comment1 ""
@@
 	5200 1400 5300 1500
 $Comp
-L VCC #PWR13
+L VCC #PWR01
 U 1 1 4F085452
 P 2600 5450
-F 0 "#PWR13" H 2600 5550 30  0001 C CNN
+F 0 "#PWR01" H 2600 5550 30  0001 C CNN
 F 1 "VCC" H 2600 5550 30  0000 C CNN
 F 2 "" H 2600 5450 60  0001 C CNN
@@
 $EndComp
 $Comp
-L VCC #PWR4
+L VCC #PWR02
 U 1 1 4F08534F
 P 1500 5450
-F 0 "#PWR4" H 1500 5550 30  0001 C CNN
+F 0 "#PWR02" H 1500 5550 30  0001 C CNN
 F 1 "VCC" H 1500 5550 30  0000 C CNN
 F 2 "" H 1500 5450 60  0001 C CNN
@@
 $EndComp
 $Comp
-L GND #PWR8
+L GND #PWR03
 U 1 1 4F08176B
 P 2100 4450
-F 0 "#PWR8" H 2100 4450 30  0001 C CNN
+F 0 "#PWR03" H 2100 4450 30  0001 C CNN
 F 1 "GND" H 2100 4380 30  0001 C CNN
 F 2 "" H 2100 4450 60  0001 C CNN
@@
 $EndComp
 $Comp
-L GND #PWR7
+L GND #PWR04
 U 1 1 4F081769
 P 1900 4450
-F 0 "#PWR7" H 1900 4450 30  0001 C CNN
+F 0 "#PWR04" H 1900 4450 30  0001 C CNN
 F 1 "GND" H 1900 4380 30  0001 C CNN
 F 2 "" H 1900 4450 60  0001 C CNN
@@
 $EndComp
 $Comp
-L VCC #PWR23
+L VCC #PWR05
 U 1 1 4ED6BD35
 P 4700 1050
-F 0 "#PWR23" H 4700 1150 30  0001 C CNN
+F 0 "#PWR05" H 4700 1150 30  0001 C CNN
 F 1 "VCC" H 4700 1150 30  0000 C CNN
 F 2 "" H 4700 1050 60  0001 C CNN
@@
 $EndComp
 $Comp
-L GND #PWR24
+L GND #PWR06
 U 1 1 4ED6BD03
 P 4700 1850
-F 0 "#PWR24" H 4700 1850 30  0001 C CNN
+F 0 "#PWR06" H 4700 1850 30  0001 C CNN
 F 1 "GND" H 4700 1780 30  0001 C CNN
 F 2 "" H 4700 1850 60  0001 C CNN
@@
 	3000 1200 3100 1300
 $Comp
-L GND #PWR1
+L GND #PWR07
 U 1 1 4ED6BB30
 P 800 3500
-F 0 "#PWR1" H 800 3500 30  0001 C CNN
+F 0 "#PWR07" H 800 3500 30  0001 C CNN
 F 1 "GND" H 800 3430 30  0001 C CNN
 F 2 "" H 800 3500 60  0001 C CNN
@@
 $EndComp
 $Comp
-L VCC #PWR12
+L VCC #PWR08
 U 1 1 4ED6BA8E
 P 2550 750
-F 0 "#PWR12" H 2550 850 30  0001 C CNN
+F 0 "#PWR08" H 2550 850 30  0001 C CNN
 F 1 "VCC" H 2550 850 30  0000 C CNN
 F 2 "" H 2550 750 60  0001 C CNN
@@
 $EndComp
 $Comp
-L GND #PWR25
+L GND #PWR09
 U 1 1 4ED6AF1D
 P 5500 7650
-F 0 "#PWR25" H 5500 7650 30  0001 C CNN
+F 0 "#PWR09" H 5500 7650 30  0001 C CNN
 F 1 "GND" H 5500 7580 30  0001 C CNN
 F 2 "" H 5500 7650 60  0001 C CNN
@@
 $EndComp
 $Comp
-L GND #PWR14
+L GND #PWR010
 U 1 1 4ED6A667
 P 2600 7350
-F 0 "#PWR14" H 2600 7350 30  0001 C CNN
+F 0 "#PWR010" H 2600 7350 30  0001 C CNN
 F 1 "GND" H 2600 7280 30  0001 C CNN
 F 2 "" H 2600 7350 60  0001 C CNN
@@
 $EndComp
 $Comp
-L GND #PWR9
+L GND #PWR011
 U 1 1 4ED6A5D7
 P 2350 7350
-F 0 "#PWR9" H 2350 7350 30  0001 C CNN
+F 0 "#PWR011" H 2350 7350 30  0001 C CNN
 F 1 "GND" H 2350 7280 30  0001 C CNN
 F 2 "" H 2350 7350 60  0001 C CNN
@@
 $EndComp
 $Comp
-L GND #PWR5
+L GND #PWR012
 U 1 1 4ED6A418
 P 1500 6250
-F 0 "#PWR5" H 1500 6250 30  0001 C CNN
+F 0 "#PWR012" H 1500 6250 30  0001 C CNN
 F 1 "GND" H 1500 6180 30  0001 C CNN
 F 2 "" H 1500 6250 60  0001 C CNN
@@
 $EndComp
 $Comp
-L VCC #PWR15
+L VCC #PWR013
 U 1 1 4EB30C92
 P 3550 2250
-F 0 "#PWR15" H 3550 2350 30  0001 C CNN
+F 0 "#PWR013" H 3550 2350 30  0001 C CNN
 F 1 "VCC" H 3550 2350 30  0000 C CNN
 F 2 "" H 3550 2250 60  0001 C CNN
@@
 $EndComp
 $Comp
-L VCC #PWR17
+L VCC #PWR014
 U 1 1 4EB30C91
 P 3650 2250
-F 0 "#PWR17" H 3650 2350 30  0001 C CNN
+F 0 "#PWR014" H 3650 2350 30  0001 C CNN
 F 1 "VCC" H 3650 2350 30  0000 C CNN
 F 2 "" H 3650 2250 60  0001 C CNN
@@
 $EndComp
 $Comp
-L VCC #PWR20
+L VCC #PWR015
 U 1 1 4EB30C90
 P 3850 2250
-F 0 "#PWR20" H 3850 2350 30  0001 C CNN
+F 0 "#PWR015" H 3850 2350 30  0001 C CNN
 F 1 "VCC" H 3850 2350 30  0000 C CNN
 F 2 "" H 3850 2250 60  0001 C CNN
@@
 $EndComp
 $Comp
-L VCC #PWR22
+L VCC #PWR016
 U 1 1 4EB30C8B
 P 3950 2250
-F 0 "#PWR22" H 3950 2350 30  0001 C CNN
+F 0 "#PWR016" H 3950 2350 30  0001 C CNN
 F 1 "VCC" H 3950 2350 30  0000 C CNN
 F 2 "" H 3950 2250 60  0001 C CNN
@@
 	5200 4050 5300 4150
 $Comp
-L GND #PWR3
+L GND #PWR017
 U 1 1 4EB2CF09
 P 1100 1900
-F 0 "#PWR3" H 1100 1900 30  0001 C CNN
+F 0 "#PWR017" H 1100 1900 30  0001 C CNN
 F 1 "GND" H 1100 1830 30  0001 C CNN
 F 2 "" H 1100 1900 60  0001 C CNN
@@
 $EndComp
 $Comp
-L VCC #PWR2
+L VCC #PWR018
 U 1 1 4EB2CED6
 P 1100 750
-F 0 "#PWR2" H 1100 850 30  0001 C CNN
+F 0 "#PWR018" H 1100 850 30  0001 C CNN
 F 1 "VCC" H 1100 850 30  0000 C CNN
 F 2 "" H 1100 750 60  0001 C CNN
@@
 $EndComp
 $Comp
-L GND #PWR21
+L GND #PWR019
 U 1 1 4E99C40C
 P 3900 7350
-F 0 "#PWR21" H 3900 7350 30  0001 C CNN
+F 0 "#PWR019" H 3900 7350 30  0001 C CNN
 F 1 "GND" H 3900 7280 30  0001 C CNN
 F 2 "" H 3900 7350 60  0001 C CNN
@@
 $EndComp
 $Comp
-L GND #PWR19
+L GND #PWR020
 U 1 1 4E99C40B
 P 3800 7350
-F 0 "#PWR19" H 3800 7350 30  0001 C CNN
+F 0 "#PWR020" H 3800 7350 30  0001 C CNN
 F 1 "GND" H 3800 7280 30  0001 C CNN
 F 2 "" H 3800 7350 60  0001 C CNN
@@
 $EndComp
 $Comp
-L GND #PWR18
+L GND #PWR021
 U 1 1 4E99C407
 P 3700 7350
-F 0 "#PWR18" H 3700 7350 30  0001 C CNN
+F 0 "#PWR021" H 3700 7350 30  0001 C CNN
 F 1 "GND" H 3700 7280 30  0001 C CNN
 F 2 "" H 3700 7350 60  0001 C CNN
@@
 $EndComp
 $Comp
-L GND #PWR16
+L GND #PWR022
 U 1 1 4E99C403
 P 3600 7350
-F 0 "#PWR16" H 3600 7350 30  0001 C CNN
+F 0 "#PWR022" H 3600 7350 30  0001 C CNN
 F 1 "GND" H 3600 7280 30  0001 C CNN
 F 2 "" H 3600 7350 60  0001 C CNN
@@
 $EndComp
 $Comp
-L GND #PWR6
+L GND #PWR023
 U 1 1 4E99B659
 P 1550 4750
-F 0 "#PWR6" H 1550 4750 30  0001 C CNN
+F 0 "#PWR023" H 1550 4750 30  0001 C CNN
 F 1 "GND" H 1550 4680 30  0001 C CNN
 F 2 "" H 1550 4750 60  0001 C CNN
@@
 $EndComp
 $Comp
-L GND #PWR11
+L GND #PWR024
 U 1 1 4E99B657
 P 2450 4750
-F 0 "#PWR11" H 2450 4750 30  0001 C CNN
+F 0 "#PWR024" H 2450 4750 30  0001 C CNN
 F 1 "GND" H 2450 4680 30  0001 C CNN
 F 2 "" H 2450 4750 60  0001 C CNN
@@
 $EndComp
 $Comp
-L GND #PWR10
+L GND #PWR025
 U 1 1 4E99B655
 P 2450 4750
-F 0 "#PWR10" H 2450 4750 30  0001 C CNN
+F 0 "#PWR025" H 2450 4750 30  0001 C CNN
 F 1 "GND" H 2450 4680 30  0001 C CNN
 F 2 "" H 2450 4750 60  0001 C CNN
@@
 GPIO3
 $Comp
-L VCC #PWR29
+L VCC #PWR026
 U 1 1 516C9166
 P 10850 3050
-F 0 "#PWR29" H 10850 3150 30  0001 C CNN
+F 0 "#PWR026" H 10850 3150 30  0001 C CNN
 F 1 "VCC" H 10850 3150 30  0000 C CNN
 F 2 "" H 10850 3050 60  0001 C CNN
@@
 Connection ~ 9500 5850
 $Comp
-L GND #PWR26
+L GND #PWR027
 U 1 1 523205C7
 P 5650 3050
-F 0 "#PWR26" H 5650 3050 30  0001 C CNN
+F 0 "#PWR027" H 5650 3050 30  0001 C CNN
 F 1 "GND" H 5650 2980 30  0001 C CNN
 F 2 "" H 5650 3050 60  0001 C CNN
@@
 $EndComp
 $Comp
-L GND #PWR28
+L GND #PWR028
 U 1 1 5260096E
 P 7750 3750
-F 0 "#PWR28" H 7750 3750 30  0001 C CNN
+F 0 "#PWR028" H 7750 3750 30  0001 C CNN
 F 1 "GND" H 7750 3680 30  0001 C CNN
 F 2 "" H 7750 3750 60  0001 C CNN
@@
 $EndComp
 $Comp
-L VCC #PWR27
+L VCC #PWR029
 U 1 1 52600A30
 P 7750 3350
-F 0 "#PWR27" H 7750 3450 30  0001 C CNN
+F 0 "#PWR029" H 7750 3450 30  0001 C CNN
 F 1 "VCC" H 7750 3450 30  0000 C CNN
 F 2 "" H 7750 3350 60  0001 C CNN
@@
 L ANYTHING H2
 U 1 1 52602196
-P 9950 900
-F 0 "H2" H 9950 950 40  0000 C CNN
-F 1 "HOLE" H 9950 850 40  0000 C CNN
-F 2 "~" H 9950 900 60  0000 C CNN
-F 3 "~" H 9950 900 60  0000 C CNN
-	1    9950 900
+P 9950 950
+F 0 "H2" H 9950 1000 40  0000 C CNN
+F 1 "HOLE" H 9950 900 40  0000 C CNN
+F 2 "~" H 9950 950 60  0000 C CNN
+F 3 "~" H 9950 950 60  0000 C CNN
+	1    9950 950
 	1    0    0    -1
 $EndComp
@@
 L ANYTHING LOGO1
 U 1 1 526023FB
-P 9950 1400
-F 0 "LOGO1" H 9950 1450 40  0000 C CNN
-F 1 "Geekhack" H 9950 1350 40  0000 C CNN
-F 2 "~" H 9950 1400 60  0000 C CNN
-F 3 "~" H 9950 1400 60  0000 C CNN
-	1    9950 1400
-	1    0    0    -1
-$EndComp
+P 10600 950
+F 0 "LOGO1" H 10600 1000 40  0000 C CNN
+F 1 "Geekhack" H 10600 900 40  0000 C CNN
+F 2 "~" H 10600 950 60  0000 C CNN
+F 3 "~" H 10600 950 60  0000 C CNN
+	1    10600 950
+	1    0    0    -1
+$EndComp
+$Comp
+L ANYTHING H3
+U 1 1 5263DA92
+P 9950 1200
+F 0 "H3" H 9950 1250 40  0000 C CNN
+F 1 "HOLE" H 9950 1150 40  0000 C CNN
+F 2 "~" H 9950 1200 60  0000 C CNN
+F 3 "~" H 9950 1200 60  0000 C CNN
+	1    9950 1200
+	1    0    0    -1
+$EndComp
+$Comp
+L ANYTHING H4
+U 1 1 5263DA98
+P 9950 1450
+F 0 "H4" H 9950 1500 40  0000 C CNN
+F 1 "HOLE" H 9950 1400 40  0000 C CNN
+F 2 "~" H 9950 1450 60  0000 C CNN
+F 3 "~" H 9950 1450 60  0000 C CNN
+	1    9950 1450
+	1    0    0    -1
+$EndComp
+$Comp
+L ANYTHING H1
+U 1 1 5263DA9E
+P 9950 700
+F 0 "H1" H 9950 750 40  0000 C CNN
+F 1 "HOLE" H 9950 650 40  0000 C CNN
+F 2 "~" H 9950 700 60  0000 C CNN
+F 3 "~" H 9950 700 60  0000 C CNN
+	1    9950 700
+	1    0    0    -1
+$EndComp
+$Comp
+L ANYTHING H5
+U 1 1 5263DAA4
+P 9950 1700
+F 0 "H5" H 9950 1750 40  0000 C CNN
+F 1 "HOLE" H 9950 1650 40  0000 C CNN
+F 2 "~" H 9950 1700 60  0000 C CNN
+F 3 "~" H 9950 1700 60  0000 C CNN
+	1    9950 1700
+	1    0    0    -1
+$EndComp

Commit message: v0.12
Parts:
- added P20: SCLM, symbol CONN_1
- added P21: SDAM, symbol CONN_1
- added R6, R7: 2.2kΩ, 0805, symbol R
- added U1: MCP23018, SSOP24, symbol MCP23018_SSOP
- C1, C2: value 22p -> 22pF; footprint (none) -> 0804; Product CL21C220JBANNNC -> VJ0805A220GXXCW1BC; Supplier TME -> (none); Supplier Symbol CL21C220JBANNNC -> (none); URL (none) -> https://www.mouser.com/Search/ProductDetail.aspx?R=VJ0805A2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; Vendor Samsung -> (none)
- C3: value 1u -> 1uF; footprint (none) -> 0805; Product CL21B105KAFNNNE -> VJ0805Y105JXQTW1BC; Supplier TME -> (none); Supplier Symbol CL21B105KAFNNNE -> (none); URL (none) -> https://www.mouser.com/Search/ProductDetail.aspx?R=VJ0805Y1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; Vendor Samsung -> (none)
- C4, C5, C6, C7: value 100n -> 0.1uF; footprint (none) -> 0805; Product CL21B104KBCNNNC -> VJ0805Y104JXXAC; Supplier TME -> (none); Supplier Symbol CL21B104KBCNNNC -> (none); URL (none) -> https://www.mouser.com/Search/ProductDetail.aspx?R=VJ0805Y1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; Vendor Samsung -> (none)
- C8: value 1u -> 1uF; footprint (none) -> 0805; Product CL21B104KBCNNNC -> VJ0805Y105JXQTW1BC; Supplier TME -> (none); Supplier Symbol CL21B104KBCNNNC -> (none); URL (none) -> https://www.mouser.com/Search/ProductDetail.aspx?R=VJ0805Y1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; Vendor Samsung -> (none)
- IC1: Supplier DigiKey -> (none); Supplier Symbol ATMEGA32U4-AU-ND -> (none); URL (none) -> https://www.mouser.com/Search/ProductDetail.aspx?R=ATMEGA32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; Vendor Atmel -> (none)
- J1: value MINI -> USB MINI-B; Product U24-05XXX-1 -> Molex 67503-1020; Supplier Alibaba -> (none); Vendor Natconn -> (none)
- R1, R2: value 22 -> 22Ω; footprint (none) -> 0805; Supplier TME -> (none); Supplier Symbol CRCW080522R0JNTABC -> (none); Vendor Vishay -> (none)
- R3, R5: value 10k -> 10kΩ; footprint (none) -> 0805; Product CRCW080510K0JNTABC -> CRCW080510K0FKEB; Supplier TME -> (none); Supplier Symbol CRCW080510K0JNTABC -> (none); URL (none) -> https://www.mouser.com/Search/ProductDetail.aspx?R=CRCW0805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; Vendor Vishay -> (none)
- RF1, RF2, RF3: value R -> kΩ; footprint (none) -> through-hole
- S0: value DTSM-6 -> ADTSMW69NVTR; Supplier TME -> (none); Supplier Symbol TACTB-64K-F -> (none); Vendor Ninigi -> (none)
- X1: value ASX3F -> 7M-16.000MAAJ-T; Product 16.00M-SMDXT324 -> 7M-16.000MAAJ-T; Supplier TME -> (none); Supplier Symbol 16.00M-SMDXT324 -> (none); URL (none) -> https://www.mouser.com/Search/ProductDetail.aspx?R=7M-16.00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; Vendor YIC -> (none)
Connections:
- net GND: now also U1.1 (GND), U1.13 (ADDR)
- net VCC: now also R6.1, R7.1, U1.10 (VCC), U1.14 (RESET)
- new net COL1: U1.17 (GPA0)
- new net COL2: U1.18 (GPA1)
- new net COL3: U1.19 (GPA2)
- new net COL4: U1.20 (GPA3)
- new net ROW1: U1.7 (GPB5)
- new net ROW2: U1.6 (GPB4)
- new net ROW3: U1.5 (GPB3)
- new net ROW4: U1.4 (GPB2)
- new net ROW5: U1.3 (GPB1)
- new net ROW6: U1.2 (GPB0)
- new net SCLM: P20.1, R6.2, U1.11 (SCL)
- new net SDAM: P21.1, R7.2, U1.12 (SDA)
- no-connect marks 12 -> 18
Other:
- note added: "Drills For 'Breakoff' \nBottom Section"
- note added: "Expansion Pins"
- note added: "Geekhack\nSilkscreen\n"
- note added: "Ground Points"
- note added: "ISP Pins"
- note added: "Mounting\nHoles"
- note added: "Resistor Values dependent upon LED value"
- note added: "S06 LED"
- note added: "S11 LED"
- note added: "S16 LED"
- note added: "Serial IO Expander"
- moved on the sheet: DF2, DF3, H1, H2, H3, H4, H5, LOGO1, M1, M10, M11, M12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

Commit message: 4x5 variant
Parts:
- removed H5, M1, M10, M11, M12, M13, M14, M15, M16, M17, M2, M3, M4, M5, M6, M7, M8, M9: HOLE, ~, symbol ANYTHING
- removed P12: ROW6, symbol CONN_1
- removed P204, P205: GND, symbol CONN_1
Connections:
- net ROW6: no longer names the net of U1.2 (GPB0)
- net row6: no longer names the net of IC1.22 ((XCK1/~CTS~)PD5)
- no-connect marks 18 -> 22
Other:
- note removed: "Drills For 'Breakoff' \nBottom Section"
